Commit message: b2_z1 update

File: low-level/resources/robots/b2_z1/urdf/b2_z1.urdf (robot description, URDF)
Before this commit: robot b2_z1_description, 26 links, 25 joints
Links:
- added link gripperStator, mass 0.52603655; collision box size=0.028 0.03 0.008; collision box size=0.028 0.03 0.008
- link FL_calf: mass 1.0 -> 0.679123; geometry collision box size=0.05 0.028 0.035; collision box size=0.10 0.0245 0.018
- link FL_hip: mass 2.0 -> 2.5294; geometry collision cylinder length=0.05 radius=0.07; visual mesh filename=../assets/FL_hip.obj scale=1 1 1
- link FL_thigh: mass 3.0 -> 7.4554; geometry collision box size=0.32 0.0445 0.054; visual mesh filename=../assets/FL_thigh.obj scale=1 1 1
- link FR_calf: mass 1.0 -> 0.679123; geometry collision box size=0.05 0.028 0.035; collision box size=0.10 0.0245 0.018
- link FR_hip: mass 2.0 -> 2.5294; geometry collision cylinder length=0.05 radius=0.07; visual mesh filename=../assets/FR_hip.obj scale=1 1 1
- link FR_thigh: mass 3.0 -> 7.4554; geometry collision box size=0.25 0.028 0.04; visual mesh filename=../assets/FR_thigh.obj scale=1 1 1
- link RL_calf: mass 1.0 -> 0.679123; geometry collision box size=0.05 0.028 0.035; collision box size=0.10 0.0245 0.018
- link RL_hip: mass 2.0 -> 2.5294; geometry collision cylinder length=0.05 radius=0.07; visual mesh filename=../assets/RL_hip.obj scale=1 1 1
- link RL_thigh: mass 3.0 -> 7.4554; geometry collision box size=0.25 0.028 0.04; visual mesh filename=../assets/RL_thigh.obj scale=1 1 1
- link RR_calf: mass 1.0 -> 0.679123; geometry collision box size=0.05 0.028 0.035; collision box size=0.10 0.0245 0.018
- link RR_hip: mass 2.0 -> 2.5294; geometry collision cylinder length=0.05 radius=0.07; visual mesh filename=../assets/RR_hip.obj scale=1 1 1
- link RR_thigh: mass 3.0 -> 7.4554; geometry collision box size=0.25 0.028 0.04; visual mesh filename=../assets/RR_thigh.obj scale=1 1 1
- link base_link: geometry collision box size=0.025 0.12 0.14; collision box size=0.04 0.12 0.14
- link gripperMover: mass 0.276213 -> 0.27621302; geometry collision box size=0.028 0.03 0.008; collision box size=0.028 0.03 0.008
- link link00: mass 0.472475 -> 0.47247481
- link link01: mass 0.6 -> 0.67332551; geometry collision cylinder length=0.102 radius=0.0325; visual mesh filename=../assets/z1_Link01.stl scale=1 1 1
- link link02: mass 0.6 -> 1.19132258; geometry collision cylinder length=0.051 radius=0.0325; collision cylinder length=0.102 radius=0.0325
- link link03: mass 0.6 -> 0.83940874; geometry collision cylinder length=0.059 radius=0.0325; collision cylinder length=0.116 radius=0.02
- link link04: mass 0.4 -> 0.56404563; geometry collision cylinder length=0.067 radius=0.0325; visual mesh filename=../assets/z1_Link04.stl scale=1 1 1
- link link05: mass 0.3 -> 0.38938492
- link link06: mass 0.3 -> 0.28875807; geometry collision cylinder length=0.051 radius=0.0325; visual mesh filename=../assets/z1_Link06.stl scale=1 1 1
Joints:
- added joint gripperStator_fixed: type fixed, parent link06, child gripperStator, origin xyz=0.051 0 0 rpy=0 0 0
- joint gripperMover_fixed: origin xyz=0.1 0 0 rpy=0 0 0 -> xyz=0.049 0 0 rpy=0 0 0; parent link06 -> gripperStator
- joint joint1: limit lower=-2.61799 upper=2.61799 effort=40 velocity=3.14 -> lower=-2.6179938779914944 upper=2.6179938779914944 effort=30 velocity=3.1415
- joint joint2: limit lower=0 upper=2.96706 effort=40 velocity=3.14 -> lower=0 upper=2.9670597283903604 effort=60 velocity=3.1415
- joint joint3: limit lower=-2.87979 upper=0 effort=20 velocity=3.14 -> lower=-2.8797932657906435 upper=0 effort=30 velocity=3.1415
- joint joint4: limit lower=-1.51844 upper=1.51844 effort=10 velocity=3.14 -> lower=-1.5184364492350666 upper=1.5184364492350666 effort=30 velocity=3.1415
- joint joint5: limit lower=-1.3439 upper=1.3439 effort=5 velocity=3.14 -> lower=-1.3439035240356338 upper=1.3439035240356338 effort=30 velocity=3.1415
- joint joint6: limit lower=-2.79253 upper=2.79253 effort=5 velocity=3.14 -> lower=-2.792526803190927 upper=2.792526803190927 effort=30 velocity=3.1415

Commit message: 调整了一个新的 urdf版本测试

File: low-level/resources/robots/b2_z1/urdf/b2_z1.urdf (robot description, URDF)
Before this commit: robot b2_z1_description, 27 links, 26 joints
Links:
- added link FL_calf_rotor, mass 0.2734; collision cylinder length=0.02 radius=0.05
- added link FL_hip_rotor, mass 0.2734; collision cylinder length=0.02 radius=0.05
- added link FL_thigh_rotor, mass 0.2734; collision cylinder length=0.02 radius=0.05
- added link FR_calf_rotor, mass 0.2734; collision cylinder length=0.02 radius=0.05
- added link FR_hip_rotor, mass 0.2734; collision cylinder length=0.02 radius=0.05
- added link FR_thigh_rotor, mass 0.2734; collision cylinder length=0.02 radius=0.05
- added link RL_calf_rotor, mass 0.2734; collision cylinder length=0.02 radius=0.05
- added link RL_hip_rotor, mass 0.2734; collision cylinder length=0.02 radius=0.05
- added link RL_thigh_rotor, mass 0.2734; collision cylinder length=0.02 radius=0.05
- added link RR_calf_rotor, mass 0.2734; collision cylinder length=0.02 radius=0.05
- added link RR_hip_rotor, mass 0.2734; collision cylinder length=0.02 radius=0.05
- added link RR_thigh_rotor, mass 0.2734; collision cylinder length=0.02 radius=0.05
- added link ee_gripper_link, mass 0.001
- added link f_dc_link, mass 4.19E-15; visual mesh filename=../assets/f_dc_link.obj
- added link f_oc_link, mass 4.19E-15
- added link head_Link, mass 3.6885; collision box size=0.04 0.12 0.14; visual mesh filename=../assets/fake_head_Link.STL
- added link imu_link, mass 4.19E-15; visual mesh filename=../assets/fake_imu_link.STL
- added link lidar_link, mass 4.19E-15; collision cylinder length=0.16 radius=0.076; visual mesh filename=../assets/unitree_ladar.obj
- added link r_dc_link, mass 4.19E-15; visual mesh filename=../assets/r_dc_link.obj
- added link r_oc_link, mass 4.19E-12
- added link tail_link, mass 0.795; collision box size=0.025 0.12 0.14; visual mesh filename=../assets/fake_tail_link.STL
- link FL_calf: mass 0.679123 -> 0.404
- link FL_foot: mass 0.08 -> 0.126
- link FL_hip: mass 2.5294 -> 2.673
- link FL_thigh: mass 7.4554 -> 4.536
- link FR_calf: mass 0.679123 -> 0.404
- link FR_foot: mass 0.08 -> 0.126
- link FR_hip: mass 2.5294 -> 2.673
- link FR_thigh: mass 7.4554 -> 4.536
- link RL_calf: mass 0.679123 -> 0.404
- link RL_foot: mass 0.08 -> 0.126
- link RL_hip: mass 2.5294 -> 2.673
- link RL_thigh: mass 7.4554 -> 4.536
- link RR_calf: mass 0.679123 -> 0.404
- link RR_foot: mass 0.08 -> 0.126
- link RR_hip: mass 2.5294 -> 2.673
- link RR_thigh: mass 7.4554 -> 4.536
- link base_link: mass 40.8426 -> 35.86; geometry collision box size=0.50 0.28 0.15; visual mesh filename=../assets/base_link.obj scale=1 1 1
Joints:
- removed joint gripperMover_fixed
- added joint FL_calf_rotor_joint: type fixed, parent FL_thigh, child FL_calf_rotor, origin xyz=0 -0.05788 0
- added joint FL_hip_rotor_joint: type fixed, parent base_link, child FL_hip_rotor, origin xyz=0.20205 0.072 0
- added joint FL_thigh_rotor_joint: type fixed, parent FL_hip, child FL_thigh_rotor, origin xyz=0 -0.00798 0
- added joint FR_calf_rotor_joint: type fixed, parent FR_thigh, child FR_calf_rotor, origin xyz=0 0.05788 0
- added joint FR_hip_rotor_joint: type fixed, parent base_link, child FR_hip_rotor, origin xyz=0.20205 -0.072 0
- added joint FR_thigh_rotor_joint: type fixed, parent FR_hip, child FR_thigh_rotor, origin xyz=0 0.00798 0
- added joint RL_calf_rotor_joint: type fixed, parent RL_thigh, child RL_calf_rotor, origin xyz=0 -0.05788 0
- added joint RL_hip_rotor_joint: type fixed, parent base_link, child RL_hip_rotor, origin xyz=-0.20205 0.072 0
- added joint RL_thigh_rotor_joint: type fixed, parent RL_hip, child RL_thigh_rotor, origin xyz=0 -0.00798 0
- added joint RR_calf_rotor_joint: type fixed, parent RR_thigh, child RR_calf_rotor, origin xyz=0 0.05788 0
- added joint RR_hip_rotor_joint: type fixed, parent base_link, child RR_hip_rotor, origin xyz=-0.20205 -0.072 0
- added joint RR_thigh_rotor_joint: type fixed, parent RR_hip, child RR_thigh_rotor, origin xyz=0 0.00798 0
- added joint ee_gripper: type fixed, parent gripperStator, child ee_gripper_link, origin xyz=0.135 0 0 rpy=0 0 0
- added joint joint_f_dc: type fixed, parent base_link, child f_dc_link, origin xyz=0.41251 0.024997 0.04765 rpy=-2.3562 0 -1.5708
- added joint joint_f_oc: type fixed, parent base_link, child f_oc_link, origin xyz=0.39079 0 -0.013433 rpy=-1.5708 0 -1.5708
- added joint joint_head: type fixed, parent base_link, child head_Link
- added joint joint_imu: type fixed, parent base_link, child imu_link, origin xyz=0 -0.02341 0.04927
- added joint joint_lidar: type fixed, parent base_link, child lidar_link, origin xyz=0.34218 0 0.17851
- added joint joint_r_dc: type fixed, parent base_link, child r_dc_link, origin xyz=-0.4081 -0.025 0.024861 rpy=-2.3557 0 1.5708
- added joint joint_r_oc: type fixed, parent base_link, child r_oc_link, origin xyz=-0.38451 0 -0.023249 rpy=-1.5708 0 1.5708
- added joint joint_tail: type fixed, parent base_link, child tail_link
- added joint z1_jointGripper: type revolute, parent gripperStator, child gripperMover, origin xyz=0.049 0 0 rpy=0 0 0, axis 0 1 0, limit lower=-1.5707963267948966 upper=0.0 effort=30.0 velocity=10.0
- joint FL_calf_joint: limit lower=-2.82 upper=-0.43 effort=300 velocity=15.0 -> lower=-2.82 upper=-0.43 effort=320 velocity=14.0
- joint FR_calf_joint: limit lower=-2.82 upper=-0.43 effort=300 velocity=15.0 -> lower=-2.82 upper=-0.43 effort=320 velocity=14.0
- joint RL_calf_joint: limit lower=-2.82 upper=-0.43 effort=300 velocity=15.0 -> lower=-2.82 upper=-0.43 effort=320 velocity=14.0
- joint RR_calf_joint: limit lower=-2.82 upper=-0.43 effort=300 velocity=15.0 -> lower=-2.82 upper=-0.43 effort=320 velocity=14.0
